File: Sys09/Sys09.kicad_pcb (KiCad board)
At the start: 2 copper layers, 103.1 x 86 mm, 25 parts, among them J1 Conn_01x40_Pin, U1 MC6809, U2 MAX708, U3 74HC00, U4 74LS27, U5 74HC00, U6 74HCT245, U7 74HCT245, U8 74HCT245, U9 74HCT245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

Commit message: Added circuits for memory and serisl
Routing:
- net /CPU/~{IRST}: track 59.8 -> 81.7 mm, vias 1 -> 0
- net /CPU/AD15: track 131.9 -> 141.0 mm
- net /CPU/AD13: track 76.6 -> 75.4 mm, vias 1 -> 0
- net /CPU/AD14: track 76.6 -> 75.4 mm, vias 1 -> 0
